File: eagle/murdock_conn.brd (EAGLE design)
At the start: 47 x 31.8 mm, 13 parts, among them IC1 4017D, X1 GPS, X2 IMU, X7 MURDOCK_STACK

Commit message: final fixes for 1st production run
Parts:
- removed IC1: 4017D, 40xx:SO16
Connections:
- removed net VDD: IC1.16
- removed net VSS: IC1.8
- net 3.3V: now also S1.3, S1.4, S2.3, S2.4, S3.3, S3.4
- net GND: no longer S1.3, S1.4, S2.3, S2.4, S3.3, S3.4
Routing:
- net 3.3V: track 27.5 -> 70.4 mm
- net GND: track 183.1 -> 148.0 mm
- net 3V3SP: track 17.4 -> 34.2 mm
- net RX: track 36.8 -> 31.0 mm
- net SDA: track 18.0 -> 23.6 mm
- net SCL: track 14.6 -> 18.7 mm
- net TX: track 31.8 -> 28.0 mm
- net SW1: track 13.9 -> 17.0 mm
- net SW2: track 44.1 -> 46.3 mm, vias 1 -> 3
- net SP1: track 4.76 -> 3.71 mm
- net SW3: track 29.7 -> 28.9 mm
- net SP2: track 13.6 -> 13.0 mm
