File: eagle/murdock_conn.sch (EAGLE design)
At the start: 13 parts, among them IC1 4017D, X1 GPS, X2 IMU, X7 MURDOCK_STACK

Commit message: final fixes for 1st production run
Parts:
- removed IC1: 4017D, 40xx:4017D
Connections:
- net 3.3V: now also S1.3, S1.4, S2.3, S2.4, S3.3, S3.4
- net GND: no longer S1.3, S1.4, S2.3, S2.4, S3.3, S3.4
Changed lines of the file:
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@@
 <part name="S1" library="switch-tact" deviceset="LSH" device="" value=""/>
 <part name="S3" library="switch-tact" deviceset="LSH" device="" value=""/>
-<part name="GND14" library="supply1" deviceset="GND" device=""/>
 <part name="X7" library="murdock" deviceset="MURDOCK_STACK" device=""/>
-<part name="IC1" library="40xx" deviceset="4017" device="D"/>
+<part name="P+3" library="SparkFun-Aesthetics" deviceset="3.3V" device=""/>
 </parts>
 <sheets>
@@
 <instance part="S1" gate="G$1" x="-10.16" y="106.68" rot="R270"/>
 <instance part="S3" gate="G$1" x="-10.16" y="91.44" rot="R270"/>
-<instance part="GND14" gate="1" x="-5.08" y="83.82" smashed="yes"/>
 <instance part="X7" gate="G$1" x="149.86" y="58.42"/>
-<instance part="IC1" gate="A" x="91.44" y="127"/>
+<instance part="P+3" gate="G$1" x="-5.08" y="86.36" smashed="yes" rot="R180">
+<attribute name="VALUE" x="-6.604" y="82.296" size="1.778" layer="96" rot="R270"/>
+</instance>
 </instances>
 <busses>
@@
 <pinref part="GND13" gate="1" pin="GND"/>
 <wire x1="30.48" y1="119.38" x2="43.18" y2="119.38" width="0.1524" layer="91"/>
+</segment>
+<segment>
+<pinref part="X7" gate="G$1" pin="GND"/>
+<wire x1="127" y1="88.9" x2="116.84" y2="88.9" width="0.1524" layer="91"/>
+<label x="116.84" y="88.9" size="1.778" layer="95"/>
+</segment>
+</net>
+<net name="5V" class="0">
+<segment>
+<pinref part="X3" gate="A" pin="3"/>
+<pinref part="U$1" gate="G$1" pin="5V"/>
+<wire x1="15.24" y1="60.96" x2="25.4" y2="60.96" width="0.1524" layer="91"/>
+</segment>
+<segment>
+<pinref part="X3" gate="A" pin="4"/>
+<pinref part="U$2" gate="G$1" pin="5V"/>
+<wire x1="43.18" y1="60.96" x2="33.02" y2="60.96" width="0.1524" layer="91"/>
+</segment>
+<segment>
+<pinref part="X4" gate="A" pin="4"/>
+<pinref part="U$3" gate="G$1" pin="5V"/>
+<wire x1="43.18" y1="45.72" x2="33.02" y2="45.72" width="0.1524" layer="91"/>
+</segment>
+<segment>
+<pinref part="X5" gate="A" pin="4"/>
+<pinref part="U$4" gate="G$1" pin="5V"/>
+<wire x1="43.18" y1="30.48" x2="33.02" y2="30.48" width="0.1524" layer="91"/>
+</segment>
+<segment>
+<pinref part="X6" gate="A" pin="4"/>
+<pinref part="U$5" gate="G$1" pin="5V"/>
+<wire x1="43.18" y1="15.24" x2="33.02" y2="15.24" width="0.1524" layer="91"/>
+</segment>
+<segment>
+<pinref part="X6" gate="A" pin="3"/>
+<pinref part="U$6" gate="G$1" pin="5V"/>
+<wire x1="15.24" y1="15.24" x2="25.4" y2="15.24" width="0.1524" layer="91"/>
+</segment>
+<segment>
+<pinref part="X5" gate="A" pin="3"/>
+<pinref part="U$7" gate="G$1" pin="5V"/>
+<wire x1="15.24" y1="30.48" x2="25.4" y2="30.48" width="0.1524" layer="91"/>
+</segment>
+<segment>
+<pinref part="X4" gate="A" pin="3"/>
+<pinref part="U$8" gate="G$1" pin="5V"/>
+<wire x1="15.24" y1="45.72" x2="25.4" y2="45.72" width="0.1524" layer="91"/>
+</segment>
+<segment>
+<pinref part="X7" gate="G$1" pin="5V"/>
+<wire x1="127" y1="83.82" x2="116.84" y2="83.82" width="0.1524" layer="91"/>
+<label x="116.84" y="83.82" size="1.778" layer="95"/>
+</segment>
+</net>
+<net name="3.3V" class="0">
+<segment>
+<pinref part="X1" gate="-3" pin="S"/>
+<pinref part="P+1" gate="G$1" pin="3.3V"/>
+<wire x1="15.24" y1="76.2" x2="20.32" y2="76.2" width="0.1524" layer="91"/>
+</segment>
+<segment>
+<pinref part="X2" gate="-3" pin="S"/>
+<pinref part="P+2" gate="G$1" pin="3.3V"/>
+<wire x1="43.18" y1="76.2" x2="48.26" y2="76.2" width="0.1524" layer="91"/>
+</segment>
+<segment>
+<pinref part="X7" gate="G$1" pin="3V3"/>
+<wire x1="167.64" y1="53.34" x2="177.8" y2="53.34" width="0.1524" layer="91"/>
+<label x="177.8" y="53.34" size="1.778" layer="95" rot="MR0"/>
 </segment>
 <segment>
@@
 <wire x1="-5.08" y1="88.9" x2="-5.08" y2="86.36" width="0.1524" layer="91"/>
 <junction x="-5.08" y="88.9"/>
-<pinref part="GND14" gate="1" pin="GND"/>
-</segment>
-<segment>
-<pinref part="X7" gate="G$1" pin="GND"/>
-<wire x1="127" y1="88.9" x2="116.84" y2="88.9" width="0.1524" layer="91"/>
-<label x="116.84" y="88.9" size="1.778" layer="95"/>
+<pinref part="P+3" gate="G$1" pin="3.3V"/>
 </segment>
 </net>
-<net name="5V" class="0">
-<segment>
-<pinref part="X3" gate="A" pin="3"/>
-<pinref part="U$1" gate="G$1" pin="5V"/>
-<wire x1="15.24" y1="60.96" x2="25.4" y2="60.96" width="0.1524" layer="91"/>
-</segment>
-<segment>
-<pinref part="X3" gate="A" pin="4"/>
-<pinref part="U$2" gate="G$1" pin="5V"/>
-<wire x1="43.18" y1="60.96" x2="33.02" y2="60.96" width="0.1524" layer="91"/>
-</segment>
-<segment>
-<pinref part="X4" gate="A" pin="4"/>
-<pinref part="U$3" gate="G$1" pin="5V"/>
-<wire x1="43.18" y1="45.72" x2="33.02" y2="45.72" width="0.1524" layer="91"/>
-</segment>
-<segment>
-<pinref part="X5" gate="A" pin="4"/>
-<pinref part="U$4" gate="G$1" pin="5V"/>
-<wire x1="43.18" y1="30.48" x2="33.02" y2="30.48" width="0.1524" layer="91"/>
-</segment>
-<segment>
-<pinref part="X6" gate="A" pin="4"/>
-<pinref part="U$5" gate="G$1" pin="5V"/>
-<wire x1="43.18" y1="15.24" x2="33.02" y2="15.24" width="0.1524" layer="91"/>
-</segment>
-<segment>
-<pinref part="X6" gate="A" pin="3"/>
-<pinref part="U$6" gate="G$1" pin="5V"/>
-<wire x1="15.24" y1="15.24" x2="25.4" y2="15.24" width="0.1524" layer="91"/>
-</segment>
-<segment>
-<pinref part="X5" gate="A" pin="3"/>
-<pinref part="U$7" gate="G$1" pin="5V"/>
-<wire x1="15.24" y1="30.48" x2="25.4" y2="30.48" width="0.1524" layer="91"/>
-</segment>
-<segment>
-<pinref part="X4" gate="A" pin="3"/>
-<pinref part="U$8" gate="G$1" pin="5V"/>
-<wire x1="15.24" y1="45.72" x2="25.4" y2="45.72" width="0.1524" layer="91"/>
-</segment>
-<segment>
-<pinref part="X7" gate="G$1" pin="5V"/>
-<wire x1="127" y1="83.82" x2="116.84" y2="83.82" width="0.1524" layer="91"/>
-<label x="116.84" y="83.82" size="1.778" layer="95"/>
-</segment>
-</net>
-<net name="3.3V" class="0">
-<segment>
-<pinref part="X1" gate="-3" pin="S"/>
-<pinref part="P+1" gate="G$1" pin="3.3V"/>
-<wire x1="15.24" y1="76.2" x2="20.32" y2="76.2" width="0.1524" layer="91"/>
-</segment>
-<segment>
-<pinref part="X2" gate="-3" pin="S"/>
-<pinref part="P+2" gate="G$1" pin="3.3V"/>
-<wire x1="43.18" y1="76.2" x2="48.26" y2="76.2" width="0.1524" layer="91"/>
-</segment>
-<segment>
-<pinref part="X7" gate="G$1" pin="3V3"/>
-<wire x1="167.64" y1="53.34" x2="177.8" y2="53.34" width="0.1524" layer="91"/>
-<label x="177.8" y="53.34" size="1.778" layer="95" rot="MR0"/>
-</segment>
-</net>
