File: eagle/murdock_mcu.brd (EAGLE design)
At the start: 47 x 31.8 mm, 17 parts, among them IC1 MPU-6050, IC2 LT1763CS8-3.3, U1 USD-SOCKETNEW, X1 USBSMD, X2 MURDOCK_STACK

Commit message: power and pwm routing
Parts:
- moved X1 11.1 mm to (24.8, 26.7)
- moved C9 0.45 mm to (18.4, 19.6)
Connections:
- new net PPM: U$1.58, X2.PPM
- new net PWM1: U$1.59, X2.PWM1
- new net PWM2: U$1.61, X2.PWM2
- new net PWM3: U$1.62, X2.PWM3
- new net PWM4: U$1.57, X2.PWM4
- new net PWM5: U$1.56, X2.PWM5
- new net PWM6: U$1.27, X2.PWM6
- new net PWM7: U$1.26, X2.PWM7
Routing:
- net +3V3: track 8.88 -> 97.7 mm, vias 0 -> 5
- net PWM1: track 0.00 -> 59.0 mm, vias 0 -> 1
- net PWM2: track 0.00 -> 56.5 mm, vias 0 -> 1
- net PWM3: track 0.00 -> 53.8 mm, vias 0 -> 1
- net PWM4: track 0.00 -> 52.5 mm, vias 0 -> 1
- net PWM5: track 0.00 -> 36.7 mm, vias 0 -> 1
- net PWM6: track 0.00 -> 22.5 mm, vias 0 -> 1
- net PPM: track 0.00 -> 17.0 mm, vias 0 -> 2
- net PWM7: track 0.00 -> 14.8 mm, vias 0 -> 1
- net GND: track 5.57 -> 16.1 mm
- net N$3: track 0.00 -> 2.42 mm
- net N$4: track 0.00 -> 2.10 mm

Commit message: more routing
Parts:
- added C12, C13: (no value), SparkFun-Capacitors:0402-CAP
- added L1: (no value), seb:X22
- added R1, R2, R3: (no value), SparkFun-Resistors:0402-RES
- moved C9 21.4 mm to (38.9, 26.1)
- moved IC1 20.1 mm to (34.3, 27.1)
- moved C2 14.2 mm to (15.6, 19.4), turned to 0 degrees
- moved C8 4.85 mm to (4.47, 18.8), turned to 90 degrees
- moved C1 4.78 mm to (12.6, 26.5), turned to 90 degrees
- moved C11 4.12 mm to (23.2, 6.80), turned to 0 degrees
- moved C10 3.25 mm to (27.5, 18.5)
- moved C4 3.25 mm to (26.4, 16.1)
- moved C3 3.25 mm to (26.1, 5.05)
- moved C7 3.25 mm to (37.2, 4.90)
- moved U$1 3.25 mm to (31.7, 10.5)
- moved C5 3.25 mm to (34.9, 18.0)
- moved IC2 2.90 mm to (6.35, 24.6)
- moved C6 2.90 mm to (7.65, 19.6)
- moved U1 2.80 mm to (6.58, 16.3)
Connections:
- new net A10: U$1.43, X2.SP1
- new net A11: R2.1, U$1.44
- new net A12: R1.1, U$1.45
- new net C7: U$1.38, X2.SP2
- new net MISO: U$1.52, U1.7
- new net MOSI: U$1.53, U1.3
- new net N$1: R2.2, X1.D-
- new net N$2: R1.2, X1.D+
- new net N$5: R3.2, U$1.5
- new net N$6: C13.2, L1.1, R3.1
- new net N$7: C12.2, L1.3, U$1.6
- new net N$8: X2.3V3_SP, X2.SW1
- new net N$9: X2.SW2, X2.SW3
- new net RX: U$1.15, X2.RX
- new net SCK: U$1.51, U1.5
- new net SD_CS: U$1.50, U1.2
- new net TX: U$1.14, X2.TX
- net GND: now also C12.1, C13.1
Routing:
- net N$8: track 0.00 -> 42.1 mm
- net N$9: track 0.00 -> 36.7 mm
- net MISO: track 0.00 -> 27.6 mm
- net MOSI: track 0.00 -> 24.3 mm
- net SCK: track 0.00 -> 23.0 mm, vias 0 -> 2
- net A10: track 0.00 -> 19.7 mm
- net SD_CS: track 0.00 -> 19.6 mm, vias 0 -> 2
- net C7: track 0.00 -> 19.0 mm
- net +3V3: track 97.7 -> 115.6 mm, vias 5 -> 7
- net RX: track 0.00 -> 17.5 mm, vias 0 -> 1
- net TX: track 0.00 -> 17.4 mm, vias 0 -> 1
- net A12: track 0.00 -> 14.1 mm
- net A11: track 0.00 -> 12.5 mm
- net N$6: track 0.00 -> 6.18 mm
- net N$7: track 0.00 -> 4.86 mm
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
Commit message: final fixes for 1st production run
Parts:
- removed C9: (no value), SparkFun-Capacitors:0402-CAP
- added C14, C16, C18: 100nF, SparkFun:0402-CAP
- added C15: 10nF, SparkFun:0402-CAP
- added C17: 2,2nF, SparkFun:0402-CAP
- added IC3: STM32F4XX_64, stm32:TQFP64
- added Q2: (no value), microbuilder:SOT23-R
- added R4, R5: (no value), SparkFun:0402-RES
- IC1: value MPU-6050 -> MPU-9150
- U$1: value STM32F4XX_64 -> (none); device stm32:TQFP64 -> seb:C3D2_LOGO_SMALL
- moved U$1 18.6 mm to (17.1, 21.9), flipped to the bottom, turned to 0 degrees
- moved X1 3.20 mm to (21.6, 26.7)
- moved R2 1.76 mm to (22.9, 20.7)
- moved C8 1.65 mm to (4.47, 20.5)
- moved C6 1.60 mm to (7.60, 21.2)
- moved R1 1.55 mm to (21.7, 20.7)
- moved C10 1.17 mm to (26.4, 18.1)
- moved IC2 1.15 mm to (6.35, 25.8)
- moved IC1 0.46 mm to (34.8, 27.3), turned to 90 degrees
Connections:
- new net INT: IC1.12
- new net LED_C: IC3.25, X2.LED_C
- new net LED_D: IC3.16, X2.LED_D
- new net LED_L: IC3.17, X2.LED_L
- new net N$10: C17.1, IC1.20
- new net SCL: IC1.23, IC3.29, R4.1, X2.SCL
- new net SDA: IC1.24, IC3.30, R5.1, X2.SDA
- new net SP_PWR: IC3.33, Q2.1
- new net SW1: IC3.55, IC3.60, X2.SW1
- new net SW2: IC3.35, X2.SW2
- new net SW3: IC3.36, X2.SW3
- net +3V3: now also C15.2, C16.1, C18.2, IC1.1, IC1.3, IC1.8, IC3.13, IC3.19, IC3.32, IC3.48, IC3.64, Q2.2, R4.2, R5.2; no longer C9.1, U$1.13, U$1.19, U$1.32, U$1.48, U$1.64
- net +5V: now also X1.VBUS
- net A10: now also IC3.43; no longer U$1.43
- net A11: now also IC3.44; no longer U$1.44
- net A12: now also IC3.45; no longer U$1.45
- net C7: now also IC3.38; no longer U$1.38
- net GND: now also C14.1, C15.1, C16.2, C17.2, C18.1, IC1.11, IC1.15, IC1.17, IC1.6, IC1.7, IC1.9, IC3.12, IC3.18, IC3.63; no longer C9.2, U$1.12, U$1.18, U$1.63
- net MISO: now also IC3.52; no longer U$1.52
- net MOSI: now also IC3.53; no longer U$1.53
- net N$3: now also IC3.31; no longer U$1.31
- net N$4: now also IC3.47; no longer U$1.47
- net N$5: now also IC3.5; no longer U$1.5
- net N$7: now also IC3.6; no longer U$1.6
- net N$8: now also Q2.3; no longer X2.SW1
- net N$9: now also C14.2, IC1.10; no longer X2.SW2, X2.SW3
- net PPM: now also IC3.23; no longer U$1.58
- net PWM1: now also IC3.58; no longer U$1.59
- net PWM2: now also IC3.59; no longer U$1.61
- net PWM3: now also IC3.62; no longer U$1.62
- net PWM4: now also IC3.61; no longer U$1.57
- net PWM5: now also IC3.22; no longer U$1.56
- net PWM6: now also IC3.27; no longer U$1.27
- net PWM7: now also IC3.26; no longer U$1.26
- net RX: now also IC3.15; no longer U$1.15
- net SCK: now also IC3.51; no longer U$1.51
- net SD_CS: now also IC3.50; no longer U$1.50
- net TX: now also IC3.14; no longer U$1.14
Routing:
- net N$8: track 42.1 -> 1.70 mm
- net SW1: track 0.00 -> 38.7 mm, vias 0 -> 2
- net SDA: track 0.00 -> 37.7 mm, vias 0 -> 3
- net +3V3: track 115.6 -> 152.6 mm, vias 7 -> 9
- net SCL: track 0.00 -> 34.8 mm, vias 0 -> 1
- net N$9: track 36.7 -> 2.16 mm
- net SW3: track 0.00 -> 25.5 mm
- net SW2: track 0.00 -> 24.7 mm
- net GND: track 18.1 -> 41.4 mm, vias 12 -> 25
- net SP_PWR: track 0.00 -> 20.7 mm
- net LED_C: track 0.00 -> 19.3 mm, vias 0 -> 1
- net +5V: track 24.1 -> 39.4 mm, vias 1 -> 2
- net LED_L: track 0.00 -> 15.2 mm
- net PWM5: track 36.2 -> 23.8 mm, vias 1 -> 2
- net LED_D: track 0.00 -> 10.6 mm
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Other:
- board text added: "MUDOCK"
- board text added: "seb@exse.net"
