File: eagle/murdock_mcu.sch (EAGLE design)
At the start: 17 parts, among them IC1 MPU-6050, IC2 LT1763CS8-3.3, U1 USD-SOCKETNEW, X1 USBSMD, X2 MURDOCK_STACK

Commit message: power and pwm routing
Connections:
- new net PPM: U$1G$3.PORTB_6, X2.PPM
- new net PWM1: U$1G$3.PORTB_7, X2.PWM1
- new net PWM2: U$1G$3.PORTB_8, X2.PWM2
- new net PWM3: U$1G$3.PORTB_9, X2.PWM3
- new net PWM4: U$1G$3.PORTB_5, X2.PWM4
- new net PWM5: U$1G$3.PORTB_4, X2.PWM5
- new net PWM6: U$1G$3.PORTB_1, X2.PWM6
- new net PWM7: U$1G$3.PORTB_0, X2.PWM7
Other:
- moved on the sheet: U$1G$2, U$1G$3
Changed lines of the file:
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@@
 <instances>
 <instance part="U$1" gate="G$1" x="-58.42" y="86.36"/>
-<instance part="U$1" gate="G$2" x="-2.54" y="86.36"/>
-<instance part="U$1" gate="G$3" x="35.56" y="86.36"/>
+<instance part="U$1" gate="G$2" x="-12.7" y="86.36"/>
+<instance part="U$1" gate="G$3" x="43.18" y="86.36"/>
 <instance part="U$1" gate="G$4" x="-2.54" y="-12.7"/>
 <instance part="U$1" gate="G$5" x="-58.42" y="142.24"/>
@@
 <instance part="+3V9" gate="G$1" x="264.16" y="45.72"/>
 <instance part="C8" gate="G$1" x="271.78" y="30.48" rot="R180"/>
-<instance part="P+1" gate="1" x="86.36" y="63.5" rot="R90"/>
+<instance part="P+1" gate="1" x="81.28" y="63.5" rot="R90"/>
 <instance part="+3V1" gate="G$1" x="149.86" y="33.02" rot="R270"/>
 <instance part="C1" gate="G$1" x="198.12" y="33.02"/>
@@
 <pinref part="X2" gate="G$1" pin="5V"/>
 <pinref part="P+1" gate="1" pin="+5V"/>
-<wire x1="88.9" y1="63.5" x2="96.52" y2="63.5" width="0.1524" layer="91"/>
+<wire x1="83.82" y1="63.5" x2="96.52" y2="63.5" width="0.1524" layer="91"/>
 </segment>
 </net>
@@
 </segment>
 </net>
+<net name="PWM1" class="0">
+<segment>
+<pinref part="X2" gate="G$1" pin="PWM1"/>
+<wire x1="96.52" y1="58.42" x2="83.82" y2="58.42" width="0.1524" layer="91"/>
+<label x="83.82" y="58.42" size="1.778" layer="95"/>
+</segment>
+<segment>
+<pinref part="U$1" gate="G$3" pin="PORTB_7"/>
+<wire x1="38.1" y1="127" x2="30.48" y2="127" width="0.1524" layer="91"/>
+<label x="30.48" y="127" size="1.778" layer="95"/>
+</segment>
+</net>
+<net name="PWM2" class="0">
+<segment>
+<pinref part="X2" gate="G$1" pin="PWM2"/>
+<wire x1="96.52" y1="53.34" x2="83.82" y2="53.34" width="0.1524" layer="91"/>
+<label x="83.82" y="53.34" size="1.778" layer="95"/>
+</segment>
+<segment>
+<pinref part="U$1" gate="G$3" pin="PORTB_8"/>
+<wire x1="38.1" y1="132.08" x2="30.48" y2="132.08" width="0.1524" layer="91"/>
+<label x="30.48" y="132.08" size="1.778" layer="95"/>
+</segment>
+</net>
+<net name="PWM4" class="0">
+<segment>
+<pinref part="X2" gate="G$1" pin="PWM4"/>
+<wire x1="96.52" y1="48.26" x2="83.82" y2="48.26" width="0.1524" layer="91"/>
+<label x="83.82" y="48.26" size="1.778" layer="95"/>
+</segment>
+<segment>
+<pinref part="U$1" gate="G$3" pin="PORTB_5"/>
+<wire x1="38.1" y1="116.84" x2="30.48" y2="116.84" width="0.1524" layer="91"/>
+<label x="30.48" y="116.84" size="1.778" layer="95"/>
+</segment>
+</net>
+<net name="PWM3" class="0">
+<segment>
+<pinref part="X2" gate="G$1" pin="PWM3"/>
+<wire x1="96.52" y1="43.18" x2="83.82" y2="43.18" width="0.1524" layer="91"/>
+<label x="83.82" y="43.18" size="1.778" layer="95"/>
+</segment>
+<segment>
+<pinref part="U$1" gate="G$3" pin="PORTB_9"/>
+<wire x1="38.1" y1="137.16" x2="30.48" y2="137.16" width="0.1524" layer="91"/>
+<label x="30.48" y="137.16" size="1.778" layer="95"/>
+</segment>
+</net>
+<net name="PWM7" class="0">
+<segment>
+<pinref part="X2" gate="G$1" pin="PWM7"/>
+<wire x1="137.16" y1="43.18" x2="149.86" y2="43.18" width="0.1524" layer="91"/>
+<label x="144.78" y="43.18" size="1.778" layer="95"/>
+</segment>
+<segment>
+<pinref part="U$1" gate="G$3" pin="PORTB_0"/>
+<wire x1="38.1" y1="91.44" x2="30.48" y2="91.44" width="0.1524" layer="91"/>
+<label x="30.48" y="91.44" size="1.778" layer="95"/>
+</segment>
+</net>
+<net name="PWM6" class="0">
+<segment>
+<pinref part="X2" gate="G$1" pin="PWM6"/>
+<wire x1="137.16" y1="63.5" x2="149.86" y2="63.5" width="0.1524" layer="91"/>
+<label x="144.78" y="63.5" size="1.778" layer="95"/>
+</segment>
+<segment>
+<pinref part="U$1" gate="G$3" pin="PORTB_1"/>
+<wire x1="38.1" y1="96.52" x2="30.48" y2="96.52" width="0.1524" layer="91"/>
+<label x="30.48" y="96.52" size="1.778" layer="95"/>
+</segment>
+</net>
+<net name="PWM5" class="0">
+<segment>
+<pinref part="X2" gate="G$1" pin="PWM5"/>
+<wire x1="137.16" y1="68.58" x2="149.86" y2="68.58" width="0.1524" layer="91"/>
+<label x="144.78" y="68.58" size="1.778" layer="95"/>
+</segment>
+<segment>
+<pinref part="U$1" gate="G$3" pin="PORTB_4"/>
+<wire x1="38.1" y1="111.76" x2="30.48" y2="111.76" width="0.1524" layer="91"/>
+<label x="30.48" y="111.76" size="1.778" layer="95"/>
+</segment>
+</net>
+<net name="PPM" class="0">
+<segment>
+<pinref part="X2" gate="G$1" pin="PPM"/>
+<wire x1="137.16" y1="38.1" x2="149.86" y2="38.1" width="0.1524" layer="91"/>
+<label x="144.78" y="38.1" size="1.778" layer="95"/>
+</segment>
+<segment>
+<pinref part="U$1" gate="G$3" pin="PORTB_6"/>
+<wire x1="38.1" y1="121.92" x2="30.48" y2="121.92" width="0.1524" layer="91"/>
+<label x="30.48" y="121.92" size="1.778" layer="95"/>
+</segment>
+</net>

Commit message: more routing
Parts:
- added C12, C13: (no value), SparkFun-Capacitors:CAP0402-CAP
- added L1: (no value), seb:X22-OSCILLATOR
- added R1, R2, R3: (no value), SparkFun-Resistors:RESISTOR0402-RES
Connections:
- new net A10: U$1G$2.PORTA_10, X2.SP1
- new net A11: R2.1, U$1G$2.PORTA_11
- new net A12: R1.1, U$1G$2.PORTA_12
- new net C7: U$1G$4.PORTC_7, X2.SP2
- new net MISO: U$1G$4.PORTC_11, U1.DO
- new net MOSI: U$1G$4.PORTC_12, U1.DI
- new net N$1: R2.2, X1.D-
- new net N$2: R1.2, X1.D+
- new net N$5: R3.2, U$1G$5.PORTH_0
- new net N$6: C13.2, L1.1, R3.1
- new net N$7: C12.2, L1.2, U$1G$5.PORTH_1
- new net N$8: X2.3V3_SP, X2.SW1
- new net N$9: X2.SW2, X2.SW3
- new net RX: U$1G$2.PORTA_1, X2.RX
- new net SCK: U$1G$4.PORTC_10, U1.SCK
- new net SD_CS: U$1G$2.PORTA_15, U1.CS
- new net TX: U$1G$2.PORTA_0, X2.TX
- net GND: now also C12.1, C13.1
Other:
- moved on the sheet: C10, C11, U$1G$1, U1

Commit message: final fixes for 1st production run
Parts:
- removed C9: (no value), SparkFun-Capacitors:CAP0402-CAP
- added C14, C16, C18: 100nF, SparkFun:CAP0402-CAP
- added C15: 10nF, SparkFun:CAP0402-CAP
- added C17: 2,2nF, SparkFun:CAP0402-CAP
- added Q2: (no value), microbuilder:MOSFET-P
- added R4, R5: (no value), SparkFun:RESISTOR0402-RES
- IC1: value MPU-6050 -> MPU-9150; device seb:MPU-6050 -> seb:MPU-9150
- renumbered U$1 to IC3
Connections:
- new net INT: IC1.12
- new net LED_C: IC3G$4.PORTC_5, X2.LED_C
- new net LED_D: IC3G$2.PORTA_2, X2.LED_D
- new net LED_L: IC3G$2.PORTA_3, X2.LED_L
- new net N$10: C17.1, IC1.20
- new net SCL: IC1.23, IC3G$3.PORTB_10, R4.1, X2.SCL
- new net SDA: IC1.24, IC3G$3.PORTB_11, R5.1, X2.SDA
- new net SP_PWR: IC3G$3.PORTB_12, Q2.G
- new net SW1: IC3G$1.BOOT0, IC3G$3.PORTB_3, X2.SW1
- new net SW2: IC3G$3.PORTB_14, X2.SW2
- new net SW3: IC3G$3.PORTB_15, X2.SW3
- net +3V3: now also C15.2, C16.1, C18.2, IC1.1, IC1.3/13, IC1.8, Q2.S, R4.2, R5.2; no longer C9.1, IC1.13
- net +5V: now also X1.VBUS
- net GND: now also C14.1, C15.1, C16.2, C17.2, C18.1, IC1.11, IC1.15/17/18, IC1.6, IC1.7, IC1.9; no longer C9.2, IC1.18
- net N$8: now also Q2.D; no longer X2.SW1
- net N$9: now also C14.2, IC1.10; no longer X2.SW2, X2.SW3
- net PPM: now also IC3G$2.PORTA_7; no longer IC3G$3.PORTB_6
- net PWM1: now also IC3G$3.PORTB_6; no longer IC3G$3.PORTB_7
- net PWM2: now also IC3G$3.PORTB_7; no longer IC3G$3.PORTB_8
- net PWM4: now also IC3G$3.PORTB_8; no longer IC3G$3.PORTB_5
- net PWM5: now also IC3G$2.PORTA_6; no longer IC3G$3.PORTB_4
Other:
- moved on the sheet: IC1
