File: eagle/murdock_conn_v2.brd (EAGLE design)
At the start: 47 x 31.8 mm, 12 parts, among them X1 GPS, X2 IMU, X7 MURDOCK_STACK

Commit message: updated stack schematic
Parts:
- moved X7 31.8 mm to (0.00, 0.00), turned to 0 degrees
Changed lines of the file:
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@@
 <?xml version="1.0" encoding="utf-8"?>
 <!DOCTYPE eagle SYSTEM "eagle.dtd">
-<eagle version="6.2">
+<eagle version="6.4">
 <drawing>
 <settings>
@@
 <layer number="21" name="tPlace" color="7" fill="1" visible="no" active="yes"/>
 <layer number="22" name="bPlace" color="7" fill="1" visible="yes" active="yes"/>
-<layer number="23" name="tOrigins" color="15" fill="1" visible="no" active="yes"/>
+<layer number="23" name="tOrigins" color="15" fill="1" visible="yes" active="yes"/>
 <layer number="24" name="bOrigins" color="15" fill="1" visible="yes" active="yes"/>
 <layer number="25" name="tNames" color="7" fill="1" visible="no" active="yes"/>
@@
 </class>
 </classes>
-<designrules>
+<designrules name="default">
 <description language="de">&lt;b&gt;EAGLE Design Rules&lt;/b&gt;
 &lt;p&gt;
@@
 <attribute name="VALUE" x="25.7175" y="13.335" size="1.27" layer="27" rot="R180"/>
 </element>
-<element name="X7" library="murdock" package="MURDOCK_STACK" value="MURDOCK_STACK" x="0" y="31.75" rot="R270"/>
+<element name="X7" library="murdock" package="MURDOCK_STACK" value="MURDOCK_STACK" x="0" y="0"/>
 </elements>
 <signals>
