File: eagle/murdock_top_v2.brd (EAGLE design)
At the start: 47 x 31.8 mm, 35 parts, among them IC1 74HC595D, IC2 74HC595D, X1 MURDOCK_STACK

Commit message: updated labels
Other:
- board text added: "BIND"
- board text added: "PPM"
- board text added: "SBUS"
- board text added: "SP1"
- board text added: "SP2"
Changed lines of the file:
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@@
 <grid distance="0.1" unitdist="mm" unit="mm" style="lines" multiple="1" display="no" altdistance="0.025" altunitdist="inch" altunit="inch"/>
 <layers>
-<layer number="1" name="Top" color="4" fill="1" visible="no" active="yes"/>
+<layer number="1" name="Top" color="4" fill="1" visible="yes" active="yes"/>
 <layer number="2" name="Route2" color="1" fill="3" visible="no" active="no"/>
 <layer number="3" name="Route3" color="4" fill="3" visible="no" active="no"/>
@@
 <layer number="14" name="Route14" color="1" fill="6" visible="no" active="no"/>
 <layer number="15" name="Route15" color="4" fill="6" visible="no" active="no"/>
-<layer number="16" name="Bottom" color="1" fill="1" visible="yes" active="yes"/>
+<layer number="16" name="Bottom" color="1" fill="1" visible="no" active="yes"/>
 <layer number="17" name="Pads" color="2" fill="1" visible="yes" active="yes"/>
 <layer number="18" name="Vias" color="2" fill="1" visible="yes" active="yes"/>
 <layer number="19" name="Unrouted" color="6" fill="1" visible="yes" active="yes"/>
 <layer number="20" name="Dimension" color="15" fill="1" visible="yes" active="yes"/>
-<layer number="21" name="tPlace" color="7" fill="1" visible="no" active="yes"/>
-<layer number="22" name="bPlace" color="7" fill="1" visible="yes" active="yes"/>
-<layer number="23" name="tOrigins" color="15" fill="1" visible="no" active="yes"/>
-<layer number="24" name="bOrigins" color="15" fill="1" visible="yes" active="yes"/>
-<layer number="25" name="tNames" color="14" fill="1" visible="no" active="yes"/>
-<layer number="26" name="bNames" color="7" fill="1" visible="yes" active="yes"/>
+<layer number="21" name="tPlace" color="7" fill="1" visible="yes" active="yes"/>
+<layer number="22" name="bPlace" color="7" fill="1" visible="no" active="yes"/>
+<layer number="23" name="tOrigins" color="15" fill="1" visible="yes" active="yes"/>
+<layer number="24" name="bOrigins" color="15" fill="1" visible="no" active="yes"/>
+<layer number="25" name="tNames" color="14" fill="1" visible="yes" active="yes"/>
+<layer number="26" name="bNames" color="7" fill="1" visible="no" active="yes"/>
 <layer number="27" name="tValues" color="7" fill="1" visible="no" active="yes"/>
 <layer number="28" name="bValues" color="7" fill="1" visible="no" active="yes"/>
-<layer number="29" name="tStop" color="12" fill="1" visible="no" active="yes"/>
-<layer number="30" name="bStop" color="7" fill="6" visible="yes" active="yes"/>
+<layer number="29" name="tStop" color="12" fill="1" visible="yes" active="yes"/>
+<layer number="30" name="bStop" color="7" fill="6" visible="no" active="yes"/>
 <layer number="31" name="tCream" color="7" fill="4" visible="no" active="yes"/>
 <layer number="32" name="bCream" color="7" fill="5" visible="no" active="yes"/>
@@
 <wire x1="12.7" y1="31.115" x2="12.7" y2="19.431" width="0.254" layer="21"/>
 <wire x1="3.865" y1="19.431" x2="12.7" y2="19.431" width="0.254" layer="21"/>
+<text x="17" y="29.2" size="0.8128" layer="21" font="vector" ratio="10">SBUS</text>
+<text x="22.5" y="26.6" size="0.8128" layer="21" font="vector" ratio="10">PPM</text>
+<text x="18.2" y="22" size="0.8128" layer="21" font="vector" ratio="10">SP1</text>
+<text x="26.7" y="22" size="0.8128" layer="21" font="vector" ratio="10">SP2</text>
+<text x="27.2" y="29.2" size="0.8128" layer="21" font="vector" ratio="10">BIND</text>
 </plain>
 <attributes>

Commit message: updated stack schematic
Parts:
- moved X1 31.8 mm to (0.00, 0.00), turned to 0 degrees
Changed lines of the file:
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@@
 <setting verticaltext="up"/>
 </settings>
-<grid distance="0.1" unitdist="mm" unit="mm" style="lines" multiple="1" display="no" altdistance="0.025" altunitdist="inch" altunit="inch"/>
+<grid distance="0.05" unitdist="mm" unit="mm" style="lines" multiple="1" display="no" altdistance="0.025" altunitdist="inch" altunit="inch"/>
 <layers>
 <layer number="1" name="Top" color="4" fill="1" visible="yes" active="yes"/>
@@
 <layer number="14" name="Route14" color="1" fill="6" visible="no" active="no"/>
 <layer number="15" name="Route15" color="4" fill="6" visible="no" active="no"/>
-<layer number="16" name="Bottom" color="1" fill="1" visible="no" active="yes"/>
+<layer number="16" name="Bottom" color="1" fill="1" visible="yes" active="yes"/>
 <layer number="17" name="Pads" color="2" fill="1" visible="yes" active="yes"/>
 <layer number="18" name="Vias" color="2" fill="1" visible="yes" active="yes"/>
@@
 <attribute name="VALUE" x="38.162" y="18.458" size="0.4064" layer="28" rot="MR90"/>
 </element>
-<element name="X1" library="murdock" package="MURDOCK_STACK" value="MURDOCK_STACK" x="0" y="31.75" smashed="yes" rot="R270"/>
+<element name="X1" library="murdock" package="MURDOCK_STACK" value="MURDOCK_STACK" x="0" y="0" smashed="yes"/>
 </elements>
 <signals>

Commit message: values
Parts:
- R1, R10, R11, R12, R13, R15, R16, R2, R3, R4, R5, R6, R7, R8, R9: value (none) -> 150R
- R14: value (none) -> 15R
Changed lines of the file:
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@@
 <attribute name="NAME" x="30.3325" y="2.2335" size="0.8128" layer="26" font="vector" ratio="10" rot="MR0"/>
 </element>
-<element name="R1" library="SparkFun-Passives" package="0402-RES" value="" x="23.4475" y="18.83" smashed="yes" rot="MR270">
+<element name="R1" library="SparkFun-Passives" package="0402-RES" value="150R" x="23.4475" y="18.83" smashed="yes" rot="MR270">
 <attribute name="NAME" x="22.649" y="19.719" size="0.8128" layer="26" font="vector" ratio="10" rot="MR270"/>
 <attribute name="VALUE" x="24.5905" y="19.9095" size="0.4064" layer="28" rot="MR270"/>
 </element>
-<element name="R2" library="SparkFun-Passives" package="0402-RES" value="" x="32.325" y="19.3025" smashed="yes" rot="MR90">
+<element name="R2" library="SparkFun-Passives" package="0402-RES" value="150R" x="32.325" y="19.3025" smashed="yes" rot="MR90">
 <attribute name="NAME" x="33.2235" y="18.8135" size="0.8128" layer="26" font="vector" ratio="10" rot="MR90"/>
 <attribute name="VALUE" x="31.182" y="18.223" size="0.4064" layer="28" rot="MR90"/>
 </element>
-<element name="R3" library="SparkFun-Passives" package="0402-RES" value="" x="31.995" y="27.4975" smashed="yes" rot="MR90">
+<element name="R3" library="SparkFun-Passives" package="0402-RES" value="150R" x="31.995" y="27.4975" smashed="yes" rot="MR90">
 <attribute name="NAME" x="32.6935" y="26.6085" size="0.8128" layer="26" font="vector" ratio="10" rot="MR90"/>
 <attribute name="VALUE" x="30.852" y="26.418" size="0.4064" layer="28" rot="MR90"/>
 </element>
-<element name="R4" library="SparkFun-Passives" package="0402-RES" value="" x="26.3875" y="30.035" smashed="yes" rot="MR270">
+<element name="R4" library="SparkFun-Passives" package="0402-RES" value="150R" x="26.3875" y="30.035" smashed="yes" rot="MR270">
 <attribute name="NAME" x="27.989" y="30.924" size="0.8128" layer="26" font="vector" ratio="10" rot="MR270"/>
 <attribute name="VALUE" x="27.5305" y="31.1145" size="0.4064" layer="28" rot="MR270"/>
 </element>
-<element name="R5" library="SparkFun-Passives" package="0402-RES" value="" x="31.565" y="16.42" smashed="yes" rot="MR90">
+<element name="R5" library="SparkFun-Passives" package="0402-RES" value="150R" x="31.565" y="16.42" smashed="yes" rot="MR90">
 <attribute name="NAME" x="32.2635" y="15.531" size="0.8128" layer="26" font="vector" ratio="10" rot="MR90"/>
 <attribute name="VALUE" x="30.422" y="15.3405" size="0.4064" layer="28" rot="MR90"/>
 </element>
-<element name="R6" library="SparkFun-Passives" package="0402-RES" value="" x="41.335" y="11.3475" smashed="yes" rot="MR90">
+<element name="R6" library="SparkFun-Passives" package="0402-RES" value="150R" x="41.335" y="11.3475" smashed="yes" rot="MR90">
 <attribute name="NAME" x="42.1335" y="10.6585" size="0.8128" layer="26" font="vector" ratio="10" rot="MR90"/>
 <attribute name="VALUE" x="40.192" y="10.268" size="0.4064" layer="28" rot="MR90"/>
 </element>
-<element name="R7" library="SparkFun-Passives" package="0402-RES" value="" x="37.17" y="29.145" smashed="yes" rot="MR180">
+<element name="R7" library="SparkFun-Passives" package="0402-RES" value="150R" x="37.17" y="29.145" smashed="yes" rot="MR180">
 <attribute name="NAME" x="36.281" y="28.4465" size="0.8128" layer="26" font="vector" ratio="10" rot="MR180"/>
 <attribute name="VALUE" x="36.0905" y="30.288" size="0.4064" layer="28" rot="MR180"/>
 </element>
-<element name="R8" library="SparkFun-Passives" package="0402-RES" value="" x="37.735" y="24.76" smashed="yes" rot="MR90">
+<element name="R8" library="SparkFun-Passives" package="0402-RES" value="150R" x="37.735" y="24.76" smashed="yes" rot="MR90">
 <attribute name="NAME" x="36.0335" y="24.171" size="0.8128" layer="26" font="vector" ratio="10" rot="MR90"/>
 <attribute name="VALUE" x="36.592" y="23.6805" size="0.4064" layer="28" rot="MR90"/>
 </element>
-<element name="R9" library="SparkFun-Passives" package="0402-RES" value="" x="13.97" y="19.685" smashed="yes" rot="MR90">
+<element name="R9" library="SparkFun-Passives" package="0402-RES" value="150R" x="13.97" y="19.685" smashed="yes" rot="MR90">
 <attribute name="NAME" x="12.3685" y="18.996" size="0.8128" layer="26" font="vector" ratio="10" rot="MR90"/>
 <attribute name="VALUE" x="12.827" y="18.6055" size="0.4064" layer="28" rot="MR90"/>
 </element>
-<element name="R10" library="SparkFun-Passives" package="0402-RES" value="" x="15.5575" y="29.21" smashed="yes" rot="MR180">
+<element name="R10" library="SparkFun-Passives" package="0402-RES" value="150R" x="15.5575" y="29.21" smashed="yes" rot="MR180">
 <attribute name="NAME" x="14.3685" y="30.8115" size="0.8128" layer="26" font="vector" ratio="10" rot="MR180"/>
 <attribute name="VALUE" x="14.478" y="30.353" size="0.4064" layer="28" rot="MR180"/>
 </element>
-<element name="R11" library="SparkFun-Passives" package="0402-RES" value="" x="9.525" y="29.21" smashed="yes" rot="MR90">
+<element name="R11" library="SparkFun-Passives" package="0402-RES" value="150R" x="9.525" y="29.21" smashed="yes" rot="MR90">
 <attribute name="NAME" x="10.2235" y="28.321" size="0.8128" layer="26" font="vector" ratio="10" rot="MR90"/>
 <attribute name="VALUE" x="8.382" y="28.1305" size="0.4064" layer="28" rot="MR90"/>
 </element>
-<element name="R12" library="SparkFun-Passives" package="0402-RES" value="" x="15.24" y="16.8275" smashed="yes" rot="MR90">
+<element name="R12" library="SparkFun-Passives" package="0402-RES" value="150R" x="15.24" y="16.8275" smashed="yes" rot="MR90">
 <attribute name="NAME" x="13.6385" y="15.7385" size="0.8128" layer="26" font="vector" ratio="10" rot="MR90"/>
 <attribute name="VALUE" x="14.097" y="15.748" size="0.4064" layer="28" rot="MR90"/>
 </element>
-<element name="R13" library="SparkFun-Passives" package="0402-RES" value="" x="4.7625" y="11.7475" smashed="yes" rot="MR90">
+<element name="R13" library="SparkFun-Passives" package="0402-RES" value="150R" x="4.7625" y="11.7475" smashed="yes" rot="MR90">
 <attribute name="NAME" x="5.561" y="10.7585" size="0.8128" layer="26" font="vector" ratio="10" rot="MR90"/>
 <attribute name="VALUE" x="3.6195" y="10.668" size="0.4064" layer="28" rot="MR90"/>
 </element>
-<element name="R14" library="SparkFun-Passives" package="0402-RES" value="" x="9.525" y="26.035" smashed="yes" rot="MR90">
+<element name="R14" library="SparkFun-Passives" package="0402-RES" value="15R" x="9.525" y="26.035" smashed="yes" rot="MR90">
 <attribute name="NAME" x="12.254" y="26.4235" size="0.8128" layer="26" font="vector" ratio="10" rot="MR0"/>
 <attribute name="VALUE" x="8.382" y="24.9555" size="0.4064" layer="28" rot="MR90"/>
 </element>
-<element name="R15" library="SparkFun-Passives" package="0402-RES" value="" x="8.89" y="23.1775" smashed="yes" rot="MR90">
+<element name="R15" library="SparkFun-Passives" package="0402-RES" value="150R" x="8.89" y="23.1775" smashed="yes" rot="MR90">
 <attribute name="NAME" x="9.5885" y="22.2885" size="0.8128" layer="26" font="vector" ratio="10" rot="MR90"/>
 <attribute name="VALUE" x="7.747" y="22.098" size="0.4064" layer="28" rot="MR90"/>
 </element>
-<element name="R16" library="SparkFun-Passives" package="0402-RES" value="" x="39.305" y="19.5375" smashed="yes" rot="MR90">
+<element name="R16" library="SparkFun-Passives" package="0402-RES" value="150R" x="39.305" y="19.5375" smashed="yes" rot="MR90">
 <attribute name="NAME" x="37.6035" y="18.4485" size="0.8128" layer="26" font="vector" ratio="10" rot="MR90"/>
 <attribute name="VALUE" x="38.162" y="18.458" size="0.4064" layer="28" rot="MR90"/>
