File: eagle/murdock_top_v2.sch (EAGLE design)
At the start: 35 parts, among them IC1 74HC595D, IC2 74HC595D, X1 MURDOCK_STACK

Commit message: values
Parts:
- R1, R10, R11, R12, R13, R15, R16, R2, R3, R4, R5, R6, R7, R8, R9: value (none) -> 150R
- R14: value (none) -> 15R
Changed lines of the file:
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@@
 <part name="P+4" library="SparkFun-Aesthetics" deviceset="3.3V" device=""/>
 <part name="P+5" library="SparkFun-Aesthetics" deviceset="3.3V" device=""/>
-<part name="R1" library="SparkFun-Passives" deviceset="RESISTOR" device="0402-RES"/>
-<part name="R2" library="SparkFun-Passives" deviceset="RESISTOR" device="0402-RES"/>
-<part name="R3" library="SparkFun-Passives" deviceset="RESISTOR" device="0402-RES"/>
-<part name="R4" library="SparkFun-Passives" deviceset="RESISTOR" device="0402-RES"/>
-<part name="R5" library="SparkFun-Passives" deviceset="RESISTOR" device="0402-RES"/>
-<part name="R6" library="SparkFun-Passives" deviceset="RESISTOR" device="0402-RES"/>
-<part name="R7" library="SparkFun-Passives" deviceset="RESISTOR" device="0402-RES"/>
-<part name="R8" library="SparkFun-Passives" deviceset="RESISTOR" device="0402-RES"/>
-<part name="R9" library="SparkFun-Passives" deviceset="RESISTOR" device="0402-RES"/>
-<part name="R10" library="SparkFun-Passives" deviceset="RESISTOR" device="0402-RES"/>
-<part name="R11" library="SparkFun-Passives" deviceset="RESISTOR" device="0402-RES"/>
-<part name="R12" library="SparkFun-Passives" deviceset="RESISTOR" device="0402-RES"/>
-<part name="R13" library="SparkFun-Passives" deviceset="RESISTOR" device="0402-RES"/>
-<part name="R14" library="SparkFun-Passives" deviceset="RESISTOR" device="0402-RES"/>
-<part name="R15" library="SparkFun-Passives" deviceset="RESISTOR" device="0402-RES"/>
-<part name="R16" library="SparkFun-Passives" deviceset="RESISTOR" device="0402-RES"/>
+<part name="R1" library="SparkFun-Passives" deviceset="RESISTOR" device="0402-RES" value="150R"/>
+<part name="R2" library="SparkFun-Passives" deviceset="RESISTOR" device="0402-RES" value="150R"/>
+<part name="R3" library="SparkFun-Passives" deviceset="RESISTOR" device="0402-RES" value="150R"/>
+<part name="R4" library="SparkFun-Passives" deviceset="RESISTOR" device="0402-RES" value="150R"/>
+<part name="R5" library="SparkFun-Passives" deviceset="RESISTOR" device="0402-RES" value="150R"/>
+<part name="R6" library="SparkFun-Passives" deviceset="RESISTOR" device="0402-RES" value="150R"/>
+<part name="R7" library="SparkFun-Passives" deviceset="RESISTOR" device="0402-RES" value="150R"/>
+<part name="R8" library="SparkFun-Passives" deviceset="RESISTOR" device="0402-RES" value="150R"/>
+<part name="R9" library="SparkFun-Passives" deviceset="RESISTOR" device="0402-RES" value="150R"/>
+<part name="R10" library="SparkFun-Passives" deviceset="RESISTOR" device="0402-RES" value="150R"/>
+<part name="R11" library="SparkFun-Passives" deviceset="RESISTOR" device="0402-RES" value="150R"/>
+<part name="R12" library="SparkFun-Passives" deviceset="RESISTOR" device="0402-RES" value="150R"/>
+<part name="R13" library="SparkFun-Passives" deviceset="RESISTOR" device="0402-RES" value="150R"/>
+<part name="R14" library="SparkFun-Passives" deviceset="RESISTOR" device="0402-RES" value="15R"/>
+<part name="R15" library="SparkFun-Passives" deviceset="RESISTOR" device="0402-RES" value="150R"/>
+<part name="R16" library="SparkFun-Passives" deviceset="RESISTOR" device="0402-RES" value="150R"/>
 <part name="GND2" library="supply1" deviceset="GND" device=""/>
 <part name="P+6" library="SparkFun-Aesthetics" deviceset="3.3V" device=""/>
