File: eagle/murdock_top_v3.sch (EAGLE design)
At the start: 35 parts, among them IC1 74HC595D, IC2 74HC595D, X1 MURDOCK_STACK

Commit message: conneced LEDs to switche 3v3
Connections:
- new net 3V3_SP: LED1.A, LED10.A, LED11.A, LED12.A, LED13.A, LED14.A, LED15.A, LED16.A, LED2.A, LED3.A, LED4.A, LED5.A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
- net 3.3V: no longer LED1.A, LED10.A, LED11.A, LED12.A, LED13.A, LED14.A, LED15.A, LED16.A, LED2.A, LED3.A, LED4.A, LED5.A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
