File: eagle/murdock_conn_v3.sch (EAGLE design)
At the start: 12 parts, among them X1 GPS, X2 IMU, X7 MURDOCK_STACK

Commit message: switch part-numbers
Parts:
- S1, S2, S3: value LSH -> min: "taster 9318" max: "taster 9319"
Changed lines of the file:
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@@
 <part name="GND12" library="supply1" deviceset="GND" device=""/>
 <part name="GND13" library="supply1" deviceset="GND" device=""/>
-<part name="S2" library="switch-tact" deviceset="LSH" device="" value=""/>
-<part name="S1" library="switch-tact" deviceset="LSH" device="" value=""/>
-<part name="S3" library="switch-tact" deviceset="LSH" device="" value=""/>
+<part name="S2" library="switch-tact" deviceset="LSH" device="" value="min: &quot;taster 9318&quot; max: &quot;taster 9319&quot;"/>
+<part name="S1" library="switch-tact" deviceset="LSH" device="" value="min: &quot;taster 9318&quot; max: &quot;taster 9319&quot;"/>
+<part name="S3" library="switch-tact" deviceset="LSH" device="" value="min: &quot;taster 9318&quot; max: &quot;taster 9319&quot;"/>
 <part name="X7" library="murdock" deviceset="MURDOCK_STACK" device=""/>
 <part name="P+3" library="SparkFun-Aesthetics" deviceset="3.3V" device=""/>
