File: eagle/murdock_conn_v4.brd (EAGLE design)
At the start: 47 x 31.8 mm, 12 parts, among them X7 MURDOCK_STACK

Commit message: v4
Parts:
- added D2: (no value), diode:SOD323-R
- added R1: 680r, SparkFun-Passives:0805
- added X1: SM06B-SRSS-TB, con-jst:SM06B-SRSS-TB
- U$9: value S4B-ZR -> ML-621S-DN; device seb:S4B-ZR -> seb:ML-621S-DN
- moved U$9 23.0 mm to (17.9, 2.50), turned to 180 degrees
Connections:
- new net BAT: D2.C, R1.2, X1.5
- new net N$1: R1.1, U$9.P
- net 3.3V: now also D2.A, X1.2; no longer U$9.3
- net GND: now also U$9.M, X1.1; no longer U$9.4
- net RX: now also X1.4; no longer U$9.2
- net TX: now also X1.3; no longer U$9.1
Routing:
- net N$1: track 0.00 -> 18.7 mm, vias 0 -> 1
- net BAT: track 0.00 -> 8.81 mm, vias 0 -> 1
- net 3.3V: track 74.0 -> 80.1 mm
- net GND: track 115.2 -> 119.7 mm
- net SW2: track 42.4 -> 45.9 mm
- net TX: track 13.6 -> 11.0 mm, vias 0 -> 1
- net RX: track 9.54 -> 10.8 mm, vias 0 -> 1
Changed lines of the file:
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@@
 </element>
 <element name="X7" library="murdock" package="MURDOCK_STACK" value="MURDOCK_STACK" x="0" y="0"/>
-<element name="U$9" library="seb" package="S4B-ZR" value="S4B-ZR" x="40.8" y="4.7275"/>
 <element name="U$12" library="seb" package="S4B-ZR" value="S4B-ZR" x="33" y="4.7275"/>
+<element name="X1" library="con-jst" package="SM06B-SRSS-TB" value="SM06B-SRSS-TB" x="39.4" y="1.9"/>
+<element name="R1" library="SparkFun-Passives" package="0805" value="680r" x="36.8" y="1.5" rot="MR180"/>
+<element name="U$9" library="seb" package="ML-621S-DN" value="ML-621S-DN" x="17.9" y="2.5" rot="R180"/>
+<element name="D2" library="diode" package="SOD323-R" value="" x="36.6" y="3.5" rot="MR0"/>
 </elements>
 <signals>
@@
 <wire x1="31.115" y1="18.115" x2="31.115" y2="16.1925" width="1.27" layer="1"/>
 <contactref element="X7" pad="GND"/>
-<contactref element="U$9" pad="4"/>
 <contactref element="U$12" pad="4"/>
 <wire x1="7.035" y1="4.7275" x2="7.035" y2="7.2" width="1.016" layer="16"/>
 <wire x1="13.285" y1="4.7275" x2="13.285" y2="6.7" width="1.016" layer="16"/>
-<wire x1="40.8" y1="4.7275" x2="40.8" y2="2.1" width="1.016" layer="16"/>
-<wire x1="33" y1="4.7275" x2="33" y2="7.8" width="1.016" layer="16"/>
+<contactref element="X1" pad="1"/>
+<wire x1="33" y1="4.7275" x2="36.9" y2="4.7275" width="0.4064" layer="1"/>
+<wire x1="36.9" y1="4.7275" x2="36.9" y2="4.875" width="0.4064" layer="1"/>
+<contactref element="U$9" pad="M"/>
+<wire x1="17.9" y1="3.24" x2="13.285" y2="3.24" width="0.6096" layer="1"/>
+<wire x1="13.285" y1="3.24" x2="13.285" y2="4.7275" width="0.6096" layer="1"/>
 </signal>
 <signal name="5V">
@@
 <wire x1="15.165" y1="11.495" x2="18.1725" y2="11.495" width="0.8128" layer="1"/>
 <wire x1="18.1725" y1="11.495" x2="28.1825" y2="11.495" width="0.8128" layer="1"/>
-<contactref element="U$9" pad="3"/>
 <contactref element="U$12" pad="3"/>
 <wire x1="31.19" y1="11.495" x2="41.2" y2="11.495" width="0.6096" layer="1"/>
 <wire x1="41.2" y1="11.495" x2="45.085" y2="11.495" width="0.6096" layer="1"/>
 <wire x1="45.085" y1="11.495" x2="45.085" y2="12.065" width="0.6096" layer="1"/>
-<wire x1="31.5" y1="4.7275" x2="31.5" y2="10.2" width="0.8128" layer="16"/>
+<wire x1="31.5" y1="4.7275" x2="31.5" y2="6.9" width="0.8128" layer="16"/>
+<wire x1="31.5" y1="6.9" x2="31.5" y2="10.2" width="0.8128" layer="16"/>
 <wire x1="31.5" y1="10.2" x2="33.365" y2="12.065" width="0.8128" layer="16"/>
 <wire x1="33.365" y1="12.065" x2="45.085" y2="12.065" width="0.8128" layer="16"/>
-<wire x1="39.3" y1="4.7275" x2="39.3" y2="3" width="0.8128" layer="1"/>
-<wire x1="39.3" y1="3" x2="31.5" y2="3" width="0.8128" layer="1"/>
-<wire x1="31.5" y1="3" x2="31.5" y2="4.7275" width="0.8128" layer="1"/>
+<contactref element="X1" pad="2"/>
+<wire x1="31.5" y1="4.7275" x2="31.5" y2="3" width="0.4064" layer="1"/>
+<wire x1="31.5" y1="3" x2="37.9" y2="3" width="0.4064" layer="1"/>
+<wire x1="37.9" y1="3" x2="37.9" y2="4.875" width="0.4064" layer="1"/>
+<contactref element="D2" pad="A"/>
+<wire x1="34.6" y1="6.9" x2="31.5" y2="6.9" width="0.4064" layer="16"/>
+<wire x1="35.5" y1="3.5" x2="34.6" y2="3.5" width="0.4064" layer="16"/>
+<wire x1="34.6" y1="3.5" x2="34.6" y2="6.9" width="0.4064" layer="16"/>
 </signal>
 <signal name="SDA">
@@
 <signal name="RX">
 <contactref element="X7" pad="RX"/>
-<contactref element="U$9" pad="2"/>
-<wire x1="37.8" y1="4.7275" x2="37.8" y2="6.985" width="0.4064" layer="16"/>
-<wire x1="37.8" y1="6.985" x2="45.085" y2="6.985" width="0.4064" layer="16"/>
+<contactref element="X1" pad="4"/>
+<wire x1="39.9" y1="4.875" x2="39.9" y2="3.1" width="0.4064" layer="1"/>
+<via x="39.9" y="3.1" extent="1-16" drill="0.4"/>
+<wire x1="39.9" y1="3.1" x2="39.9" y2="6.985" width="0.4064" layer="16"/>
+<wire x1="39.9" y1="6.985" x2="45.085" y2="6.985" width="0.4064" layer="16"/>
 </signal>
 <signal name="TX">
 <contactref element="X7" pad="TX"/>
-<contactref element="U$9" pad="1"/>
-<wire x1="36.3" y1="4.7275" x2="36.3" y2="9.525" width="0.4064" layer="16"/>
-<wire x1="36.3" y1="9.525" x2="45.085" y2="9.525" width="0.4064" layer="16"/>
+<contactref element="X1" pad="3"/>
+<wire x1="38.9" y1="4.875" x2="38.9" y2="7" width="0.4064" layer="1"/>
+<wire x1="38.9" y1="7" x2="38.8" y2="7" width="0.4064" layer="1"/>
+<via x="38.8" y="7" extent="1-16" drill="0.4"/>
+<wire x1="38.8" y1="7" x2="38.8" y2="9.525" width="0.4064" layer="16"/>
+<wire x1="38.8" y1="9.525" x2="45.085" y2="9.525" width="0.4064" layer="16"/>
 </signal>
 <signal name="PWM1">
@@
 <wire x1="31.18" y1="7.015" x2="31.18" y2="7.2375" width="0.4064" layer="1"/>
 <contactref element="X7" pad="SW2"/>
-<wire x1="30.11" y1="9.49" x2="4.48" y2="9.49" width="0.4064" layer="1"/>
+<wire x1="30.11" y1="9.49" x2="29.6" y2="9.49" width="0.4064" layer="1"/>
+<wire x1="29.6" y1="9.49" x2="4.48" y2="9.49" width="0.4064" layer="1"/>
 <wire x1="4.48" y1="9.49" x2="1.905" y2="12.065" width="0.4064" layer="1"/>
 <wire x1="30.11" y1="9.49" x2="31.18" y2="8.42" width="0.4064" layer="1"/>
 <wire x1="31.18" y1="8.42" x2="31.18" y2="7.015" width="0.4064" layer="1"/>
-<wire x1="31.18" y1="7.015" x2="41.2" y2="7.015" width="0.4064" layer="1"/>
+<wire x1="41.2" y1="7.015" x2="41.2" y2="8.5" width="0.4064" layer="1"/>
+<wire x1="41.2" y1="8.5" x2="40.2" y2="9.5" width="0.4064" layer="1"/>
+<wire x1="40.2" y1="9.5" x2="29.61" y2="9.5" width="0.4064" layer="1"/>
+<wire x1="29.61" y1="9.5" x2="29.6" y2="9.49" width="0.4064" layer="1"/>
 </signal>
 <signal name="SW1">
@@
 <wire x1="5.145" y1="7.015" x2="15.165" y2="7.015" width="0.4064" layer="1"/>
 </signal>
+<signal name="BAT">
+<contactref element="X1" pad="5"/>
+<contactref element="R1" pad="2"/>
+<wire x1="40.9" y1="4.875" x2="40.9" y2="3.6" width="0.4064" layer="1"/>
+<wire x1="40.9" y1="3.6" x2="41.4" y2="3.1" width="0.4064" layer="1"/>
+<via x="41.4" y="3.1" extent="1-16" drill="0.4"/>
+<wire x1="41.4" y1="3.1" x2="41.4" y2="2.3" width="0.4064" layer="16"/>
+<wire x1="41.4" y1="2.3" x2="40.6" y2="1.5" width="0.4064" layer="16"/>
+<wire x1="40.6" y1="1.5" x2="37.7" y2="1.5" width="0.4064" layer="16"/>
+<contactref element="D2" pad="C"/>
+<wire x1="37.7" y1="1.5" x2="37.7" y2="3.5" width="0.4064" layer="16"/>
+</signal>
+<signal name="N$1">
+<contactref element="R1" pad="1"/>
+<contactref element="U$9" pad="P"/>
+<wire x1="17.9" y1="1.76" x2="19.7" y2="1.76" width="0.4064" layer="1"/>
+<wire x1="19.7" y1="1.76" x2="19.7" y2="1.3" width="0.4064" layer="1"/>
+<via x="19.7" y="1.3" extent="1-16" drill="0.4"/>
+<wire x1="19.7" y1="1.3" x2="35.9" y2="1.3" width="0.4064" layer="16"/>
+<wire x1="35.9" y1="1.3" x2="35.9" y2="1.5" width="0.4064" layer="16"/>
+</signal>
 </signals>
