File: eagle/murdock_top_v4.brd (EAGLE design)
At the start: 47 x 31.8 mm, 35 parts, among them IC1 74HC595D, IC2 74HC595D, X1 MURDOCK_STACK

Commit message: v4
Parts:
- moved R4 1.01 mm to (27.1, 30.7), turned to 0 degrees
- turned LED12 to 90 degrees
Connections:
- new net 5V: LED1.A, LED10.A, LED11.A, LED12.A, LED13.A, LED14.A, LED15.A, LED16.A, LED2.A, LED3.A, LED4.A, LED5.A, LED6.A, LED7.A, LED8.A, LED9.A, X1.5V
- net 3V3_SP: no longer LED1.A, LED10.A, LED11.A, LED12.A, LED13.A, LED14.A, LED15.A, LED16.A, LED2.A, LED3.A, LED4.A, LED5.A, LED6.A, LED7.A, LED8.A, LED9.A
Routing:
- net 3V3_SP: track 105.9 -> 0.00 mm, vias 2 -> 0
- net 5V: track 0.00 -> 102.8 mm, vias 0 -> 2
- net N$5: track 1.09 -> 3.19 mm
- net Q3: track 30.3 -> 28.9 mm
