File: eagle/murdock_top_v4.sch (EAGLE design)
At the start: 35 parts, among them IC1 74HC595D, IC2 74HC595D, X1 MURDOCK_STACK

Commit message: v4
Connections:
- new net 5V: LED1.A, LED10.A, LED11.A, LED12.A, LED13.A, LED14.A, LED15.A, LED16.A, LED2.A, LED3.A, LED4.A, LED5.A, LED6.A, LED7.A, LED8.A, LED9.A, X1.5V
- net 3V3_SP: no longer LED1.A, LED10.A, LED11.A, LED12.A, LED13.A, LED14.A, LED15.A, LED16.A, LED2.A, LED3.A, LED4.A, LED5.A, LED6.A, LED7.A, LED8.A, LED9.A
Changed lines of the file:
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@@
 <label x="106.68" y="53.34" size="1.778" layer="95"/>
+</segment>
+</net>
+<net name="5V" class="0">
+<segment>
+<pinref part="X1" gate="G$1" pin="5V"/>
+<wire x1="119.38" y1="78.74" x2="111.76" y2="78.74" width="0.1524" layer="91"/>
+</segment>
+<segment>
+<pinref part="LED16" gate="G$1" pin="A"/>
+<pinref part="LED15" gate="G$1" pin="A"/>
+<wire x1="27.94" y1="43.18" x2="27.94" y2="50.8" width="0.1524" layer="91"/>
+<pinref part="LED14" gate="G$1" pin="A"/>
+<wire x1="27.94" y1="50.8" x2="27.94" y2="58.42" width="0.1524" layer="91"/>
+<junction x="27.94" y="50.8"/>
+<pinref part="LED13" gate="G$1" pin="A"/>
+<wire x1="27.94" y1="58.42" x2="27.94" y2="66.04" width="0.1524" layer="91"/>
+<junction x="27.94" y="58.42"/>
+<pinref part="LED12" gate="G$1" pin="A"/>
+<wire x1="27.94" y1="66.04" x2="27.94" y2="73.66" width="0.1524" layer="91"/>
+<junction x="27.94" y="66.04"/>
+<pinref part="LED11" gate="G$1" pin="A"/>
+<wire x1="27.94" y1="73.66" x2="27.94" y2="81.28" width="0.1524" layer="91"/>
+<junction x="27.94" y="73.66"/>
+<pinref part="LED10" gate="G$1" pin="A"/>
+<wire x1="27.94" y1="81.28" x2="27.94" y2="88.9" width="0.1524" layer="91"/>
+<junction x="27.94" y="81.28"/>
+<pinref part="LED9" gate="G$1" pin="A"/>
+<wire x1="27.94" y1="88.9" x2="27.94" y2="96.52" width="0.1524" layer="91"/>
+<junction x="27.94" y="88.9"/>
+<wire x1="27.94" y1="96.52" x2="27.94" y2="101.6" width="0.1524" layer="91"/>
+<junction x="27.94" y="96.52"/>
+<label x="25.4" y="101.6" size="1.778" layer="95"/>
 </segment>
 <segment>
@@
 <label x="-58.42" y="101.6" size="1.778" layer="95"/>
 </segment>
-<segment>
-<pinref part="LED16" gate="G$1" pin="A"/>
-<pinref part="LED15" gate="G$1" pin="A"/>
-<wire x1="27.94" y1="43.18" x2="27.94" y2="50.8" width="0.1524" layer="91"/>
-<pinref part="LED14" gate="G$1" pin="A"/>
-<wire x1="27.94" y1="50.8" x2="27.94" y2="58.42" width="0.1524" layer="91"/>
-<junction x="27.94" y="50.8"/>
-<pinref part="LED13" gate="G$1" pin="A"/>
-<wire x1="27.94" y1="58.42" x2="27.94" y2="66.04" width="0.1524" layer="91"/>
-<junction x="27.94" y="58.42"/>
-<pinref part="LED12" gate="G$1" pin="A"/>
-<wire x1="27.94" y1="66.04" x2="27.94" y2="73.66" width="0.1524" layer="91"/>
-<junction x="27.94" y="66.04"/>
-<pinref part="LED11" gate="G$1" pin="A"/>
-<wire x1="27.94" y1="73.66" x2="27.94" y2="81.28" width="0.1524" layer="91"/>
-<junction x="27.94" y="73.66"/>
-<pinref part="LED10" gate="G$1" pin="A"/>
-<wire x1="27.94" y1="81.28" x2="27.94" y2="88.9" width="0.1524" layer="91"/>
-<junction x="27.94" y="81.28"/>
-<pinref part="LED9" gate="G$1" pin="A"/>
-<wire x1="27.94" y1="88.9" x2="27.94" y2="96.52" width="0.1524" layer="91"/>
-<junction x="27.94" y="88.9"/>
-<wire x1="27.94" y1="96.52" x2="27.94" y2="101.6" width="0.1524" layer="91"/>
-<junction x="27.94" y="96.52"/>
-<label x="25.4" y="101.6" size="1.778" layer="95"/>
-</segment>
 </net>
