File: eagle/murdock_mcu_v4.brd (EAGLE design)
At the start: 47 x 31.8 mm, 40 parts, among them IC1 MPU-9150, IC2 LT1763CS8-3.3, IC3 STM32F4XX_64, IC4 BMP085, IC5 24LC16BSN, T1 PFET, T2 BC817, U1 USD-SOCKETNEW, X2 MURDOCK_STACK

Commit message: v4
Parts:
- U$1: value (none) -> MAKE-DD_LOGO; device seb:C3D2_LOGO_SMALL -> seb:MAKE-DD_LOGO
- moved U$1 1.10 mm to (18.2, 22.6)
Changed lines of the file:
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@@
 <layer number="28" name="bValues" color="7" fill="1" visible="no" active="yes"/>
 <layer number="29" name="tStop" color="7" fill="3" visible="yes" active="yes"/>
-<layer number="30" name="bStop" color="7" fill="6" visible="no" active="yes"/>
+<layer number="30" name="bStop" color="7" fill="6" visible="yes" active="yes"/>
 <layer number="31" name="tCream" color="7" fill="4" visible="no" active="yes"/>
 <layer number="32" name="bCream" color="7" fill="5" visible="no" active="yes"/>
@@
 <attribute name="VALUE" x="36.293" y="21.9205" size="0.4064" layer="27" rot="R90"/>
 </element>
-<element name="U$1" library="seb" package="C3D2_LOGO_SMALL" value="" x="17.1" y="22.55" rot="MR0"/>
 <element name="IC4" library="SparkFun-Sensors" package="BMP085" value="BMP085" x="26" y="26.7" smashed="yes" rot="R270"/>
 <element name="JP1" library="SparkFun-Connectors" package="USB-MICROB" value="USB-MICROB" x="17.5" y="30.3" smashed="yes" rot="R180">
@@
 <attribute name="VALUE" x="41.8795" y="2.543" size="0.4064" layer="27" rot="R180"/>
 </element>
+<element name="U$1" library="seb" package="MAKE-DD_LOGO" value="MAKE-DD_LOGO" x="18.2" y="22.6" rot="MR0"/>
 </elements>
 <signals>
@@
 <wire x1="6.95" y1="25.2" x2="9.45" y2="25.2" width="0.4064" layer="1"/>
 <via x="16.85" y="20.85" extent="1-16" drill="0.6"/>
-<via x="29.95" y="14.35" extent="1-16" drill="0.6"/>
+<via x="30.15" y="14.15" extent="1-16" drill="0.6"/>
 <via x="42.05" y="30.05" extent="1-16" drill="0.6"/>
 <via x="21.5" y="17.55" extent="1-16" drill="0.6"/>
@@
 <wire x1="39.0025" y1="12.2475" x2="37.3025" y2="12.2475" width="0.3048" layer="1"/>
 <via x="19.6" y="9.65" extent="1-16" drill="0.6"/>
-<via x="23.95" y="21.35" extent="1-16" drill="0.6"/>
+<via x="23.95" y="20.75" extent="1-16" drill="0.6"/>
 <via x="13.35" y="28.4" extent="1-16" drill="0.6"/>
 <via x="12.45" y="26.1" extent="1-16" drill="0.6"/>

Commit message: minor stuff
Parts:
- added C19, C20: 2.2µF, SparkFun-Capacitors:0805
- added C9: 100nF, SparkFun:0402-CAP
- moved C16 0.92 mm to (37.5, 30.4), turned to 0 degrees
- moved C14 0.73 mm to (39.4, 27.1)
- moved JP1 0.50 mm to (17.0, 30.3)
Connections:
- new net N$14: IC3.54
- net +3V3: now also C20.2, C9.1
- net +5V: now also C19.2
- net GND: now also C19.1, C20.1, C9.2
- net INT: now also IC3.28
Routing:
- net INT: track 0.00 -> 27.9 mm, vias 0 -> 2
- net GND: track 49.4 -> 52.2 mm
- net +3V3: track 196.1 -> 197.6 mm
- net N$9: track 2.16 -> 2.74 mm
