File: eagle/murdock_mcu_v4.sch (EAGLE design)
At the start: 39 parts, among them IC1 MPU-9150, IC2 LT1763CS8-3.3, IC3 STM32F4XX_64, IC4 BMP085, IC5 24LC16BSN, T1 PFET, T2 BC817, U1 USD-SOCKETNEW, X2 MURDOCK_STACK

Commit message: v4
Parts:
- added U$1: MAKE-DD_LOGO, seb:MAKE-DD_LOGO
Changed lines of the file:
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@@
 <part name="R11" library="SparkFun" deviceset="RESISTOR" device="0402-RES" value="4k7"/>
 <part name="+3V15" library="supply1" deviceset="+3V3" device=""/>
+<part name="U$1" library="seb" deviceset="MAKE-DD_LOGO" device=""/>
 </parts>
 <sheets>
@@
 <instance part="R11" gate="G$1" x="167.64" y="17.78" rot="R90"/>
 <instance part="+3V15" gate="G$1" x="167.64" y="35.56"/>
+<instance part="U$1" gate="G$1" x="284.48" y="-22.86"/>
 </instances>
 <busses>

Commit message: minor stuff
Parts:
- added C19, C20: 2.2µF, SparkFun-Capacitors:CAP0805
- added C9: 100nF, SparkFun:CAP0402-CAP
Connections:
- new net N$14: IC3G$5.PORTD_2
- net +3V3: now also C20.2, C9.1
- net +5V: now also C19.2
- net GND: now also C19.1, C20.1, C9.2
- net INT: now also IC3G$3.PORTB_2
Other:
- moved on the sheet: IC3G$5
Changed lines of the file:
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@@
 <part name="+3V15" library="supply1" deviceset="+3V3" device=""/>
 <part name="U$1" library="seb" deviceset="MAKE-DD_LOGO" device=""/>
+<part name="C9" library="SparkFun" deviceset="CAP" device="0402-CAP" value="100nF"/>
+<part name="GND31" library="supply1" deviceset="GND" device=""/>
+<part name="C19" library="SparkFun-Capacitors" deviceset="CAP" device="0805" value="2.2µF"/>
+<part name="C20" library="SparkFun-Capacitors" deviceset="CAP" device="0805" value="2.2µF"/>
 </parts>
 <sheets>
@@
 <instance part="IC3" gate="G$3" x="43.18" y="86.36"/>
 <instance part="IC3" gate="G$4" x="-2.54" y="-12.7"/>
-<instance part="IC3" gate="G$5" x="-58.42" y="142.24"/>
+<instance part="IC3" gate="G$5" x="-55.88" y="142.24"/>
 <instance part="U1" gate="G$1" x="58.42" y="30.48"/>
 <instance part="X2" gate="G$1" x="119.38" y="38.1"/>
@@
 <instance part="+3V15" gate="G$1" x="167.64" y="35.56"/>
 <instance part="U$1" gate="G$1" x="284.48" y="-22.86"/>
+<instance part="C9" gate="G$1" x="332.74" y="154.94"/>
+<instance part="GND31" gate="1" x="332.74" y="149.86"/>
+<instance part="C19" gate="G$1" x="205.74" y="33.02" rot="R180"/>
+<instance part="C20" gate="G$1" x="284.48" y="33.02" rot="R180"/>
 </instances>
 <busses>
@@
 <wire x1="223.52" y1="22.86" x2="226.06" y2="22.86" width="0.1524" layer="91"/>
 <wire x1="226.06" y1="22.86" x2="226.06" y2="27.94" width="0.1524" layer="91"/>
-<wire x1="220.98" y1="22.86" x2="198.12" y2="22.86" width="0.1524" layer="91"/>
+<wire x1="220.98" y1="22.86" x2="205.74" y2="22.86" width="0.1524" layer="91"/>
+<wire x1="205.74" y1="22.86" x2="198.12" y2="22.86" width="0.1524" layer="91"/>
 <wire x1="198.12" y1="22.86" x2="198.12" y2="27.94" width="0.1524" layer="91"/>
 <wire x1="198.12" y1="22.86" x2="190.5" y2="22.86" width="0.1524" layer="91"/>
@@
 <pinref part="C2" gate="G$1" pin="-"/>
 <junction x="256.54" y="27.94"/>
+<pinref part="C19" gate="G$1" pin="1"/>
+<wire x1="205.74" y1="27.94" x2="205.74" y2="22.86" width="0.1524" layer="91"/>
+<junction x="205.74" y="22.86"/>
+<pinref part="C20" gate="G$1" pin="1"/>
+<wire x1="271.78" y1="27.94" x2="284.48" y2="27.94" width="0.1524" layer="91"/>
+<junction x="271.78" y="27.94"/>
 </segment>
 <segment>
@@
 <pinref part="T2" gate="G$1" pin="E"/>
 <pinref part="GND30" gate="1" pin="GND"/>
+</segment>
+<segment>
+<pinref part="C9" gate="G$1" pin="2"/>
+<pinref part="GND31" gate="1" pin="GND"/>
 </segment>
 </net>
@@
 <pinref part="C2" gate="G$1" pin="+"/>
 <junction x="256.54" y="35.56"/>
+<pinref part="C20" gate="G$1" pin="2"/>
+<wire x1="271.78" y1="35.56" x2="284.48" y2="35.56" width="0.1524" layer="91"/>
+<junction x="271.78" y="35.56"/>
 </segment>
 <segment>
@@
 <pinref part="IC4" gate="G$1" pin="VDDA"/>
 <pinref part="+3V12" gate="G$1" pin="+3V3"/>
+<pinref part="C9" gate="G$1" pin="1"/>
+<junction x="332.74" y="160.02"/>
+<pinref part="C9" gate="G$1" pin="1"/>
 </segment>
 <segment>
@@
 <wire x1="208.28" y1="35.56" x2="208.28" y2="40.64" width="0.1524" layer="91"/>
 <wire x1="208.28" y1="40.64" x2="210.82" y2="40.64" width="0.1524" layer="91"/>
-<wire x1="208.28" y1="40.64" x2="198.12" y2="40.64" width="0.1524" layer="91"/>
+<wire x1="208.28" y1="40.64" x2="205.74" y2="40.64" width="0.1524" layer="91"/>
+<wire x1="205.74" y1="40.64" x2="198.12" y2="40.64" width="0.1524" layer="91"/>
 <wire x1="198.12" y1="40.64" x2="198.12" y2="35.56" width="0.1524" layer="91"/>
 <wire x1="198.12" y1="40.64" x2="190.5" y2="40.64" width="0.1524" layer="91"/>
@@
 <pinref part="P+3" gate="1" pin="+5V"/>
 <pinref part="C1" gate="G$1" pin="+"/>
+<pinref part="C19" gate="G$1" pin="2"/>
+<wire x1="205.74" y1="35.56" x2="205.74" y2="40.64" width="0.1524" layer="91"/>
+<junction x="205.74" y="40.64"/>
 </segment>
 <segment>
@@
 <wire x1="137.16" y1="43.18" x2="149.86" y2="43.18" width="0.1524" layer="91"/>
 <label x="144.78" y="43.18" size="1.778" layer="95"/>
+<wire x1="137.16" y1="43.18" x2="149.86" y2="43.18" width="0.1524" layer="91"/>
 </segment>
 <segment>
@@
 <pinref part="IC3" gate="G$5" pin="PORTH_0"/>
 <pinref part="R3" gate="G$1" pin="2"/>
+<wire x1="-60.96" y1="147.32" x2="-63.5" y2="147.32" width="0.1524" layer="91"/>
 </segment>
 </net>
@@
 <pinref part="IC3" gate="G$5" pin="PORTH_1"/>
 <pinref part="L1" gate="G$1" pin="2"/>
-<wire x1="-63.5" y1="152.4" x2="-76.2" y2="152.4" width="0.1524" layer="91"/>
+<wire x1="-60.96" y1="152.4" x2="-76.2" y2="152.4" width="0.1524" layer="91"/>
 <pinref part="C12" gate="G$1" pin="2"/>
 <wire x1="-76.2" y1="152.4" x2="-81.28" y2="152.4" width="0.1524" layer="91"/>
@@
 <net name="INT" class="0">
 <segment>
-<wire x1="259.08" y1="177.8" x2="279.4" y2="177.8" width="0.1524" layer="91"/>
-<wire x1="279.4" y1="177.8" x2="281.94" y2="177.8" width="0.1524" layer="91"/>
+<wire x1="259.08" y1="177.8" x2="281.94" y2="177.8" width="0.1524" layer="91"/>
 <wire x1="281.94" y1="177.8" x2="281.94" y2="185.42" width="0.1524" layer="91"/>
 <wire x1="281.94" y1="185.42" x2="304.8" y2="185.42" width="0.1524" layer="91"/>
 <pinref part="IC1" gate="G$1" pin="12"/>
 <label x="292.1" y="185.42" size="1.778" layer="95"/>
+<wire x1="30.48" y1="101.6" x2="38.1" y2="101.6" width="0.1524" layer="91"/>
+<label x="30.48" y="101.6" size="1.778" layer="95"/>
+<pinref part="IC3" gate="G$3" pin="PORTB_2"/>
 </segment>
 </net>
@@
 </segment>
 </net>
+<net name="N$14" class="0">
+<segment>
+<pinref part="IC3" gate="G$5" pin="PORTD_2"/>
+<wire x1="-60.96" y1="162.56" x2="-63.5" y2="162.56" width="0.1524" layer="91"/>
+</segment>
+</net>
