File: eagle/v2/murdock_conn_v2.brd (EAGLE design)
At the start: 47 x 31.8 mm, 12 parts, among them X1 GPS, X2 IMU, X7 MURDOCK_STACK

Commit message: switch part-numbers
Parts:
- S1, S2, S3: value (none) -> min: "taster 9318" max: "taster 9319"
Changed lines of the file:
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@@
 <element name="U$10" library="seb" package="S3B-ZR" value="S3B-ZR" x="6.985" y="4.1275" smashed="yes" rot="MR0"/>
 <element name="U$11" library="seb" package="S3B-ZR" value="S3B-ZR" x="13.335" y="4.1275" smashed="yes" rot="MR0"/>
-<element name="S2" library="switch-tact" package="LSH" value="" x="36.195" y="8.255" smashed="yes" rot="R180">
+<element name="S2" library="switch-tact" package="LSH" value="min: &quot;taster 9318&quot; max: &quot;taster 9319&quot;" x="36.195" y="8.255" smashed="yes" rot="R180">
 <attribute name="VALUE" x="38.735" y="13.335" size="1.27" layer="27" rot="R180"/>
 </element>
-<element name="S1" library="switch-tact" package="LSH" value="" x="10.16" y="8.255" smashed="yes" rot="R180">
+<element name="S1" library="switch-tact" package="LSH" value="min: &quot;taster 9318&quot; max: &quot;taster 9319&quot;" x="10.16" y="8.255" smashed="yes" rot="R180">
 <attribute name="VALUE" x="12.7" y="13.335" size="1.27" layer="27" rot="R180"/>
 </element>
-<element name="S3" library="switch-tact" package="LSH" value="" x="23.1775" y="8.255" smashed="yes" rot="R180">
+<element name="S3" library="switch-tact" package="LSH" value="min: &quot;taster 9318&quot; max: &quot;taster 9319&quot;" x="23.1775" y="8.255" smashed="yes" rot="R180">
 <attribute name="VALUE" x="25.7175" y="13.335" size="1.27" layer="27" rot="R180"/>
 </element>
