File: eagle/v2/murdock_top_v2.brd (EAGLE design)
At the start: 47 x 31.8 mm, 35 parts, among them IC1 74HC595D, IC2 74HC595D, X1 MURDOCK_STACK

Commit message: merge
Connections:
- net Q0 renamed S
- net Q1 renamed E
- net Q2 renamed NE
- net Q3 renamed N
- net Q4 renamed SE
- net Q5 renamed SETUP
- net Q6 renamed MAG_CAL
- net Q7 renamed GYRO_CAL
- net QA renamed STICK_CAL
- net QB renamed RC_OK
- net QC renamed GPS_OK
- net QD renamed MODE
- net QE renamed SW
- net QF renamed AUX_OK
- net QG renamed NW
- net QH renamed W
Changed lines of the file:
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@@
 <?xml version="1.0" encoding="utf-8"?>
 <!DOCTYPE eagle SYSTEM "eagle.dtd">
-<eagle version="6.4">
+<eagle version="6.3">
 <drawing>
 <settings>
@@
 <wire x1="23.8125" y1="10.4775" x2="26.4541" y2="10.4775" width="0.4064" layer="16"/>
 </signal>
-<signal name="QA">
+<signal name="STICK_CAL">
 <contactref element="IC1" pad="15"/>
 <contactref element="R16" pad="1"/>
@@
 <wire x1="39.305" y1="17.68" x2="39.33" y2="17.655" width="0.4064" layer="16"/>
 </signal>
-<signal name="QB">
+<signal name="RC_OK">
 <contactref element="R15" pad="1"/>
 <contactref element="IC1" pad="1"/>
@@
 <wire x1="9.2075" y1="22.21" x2="8.89" y2="22.5275" width="0.4064" layer="16"/>
 </signal>
-<signal name="QC">
+<signal name="GPS_OK">
 <contactref element="R14" pad="1"/>
 <contactref element="IC1" pad="2"/>
@@
 <wire x1="10.16" y1="24.75" x2="9.525" y2="25.385" width="0.4064" layer="16"/>
 </signal>
-<signal name="QD">
+<signal name="MODE">
 <contactref element="R13" pad="1"/>
 <contactref element="IC1" pad="3"/>
@@
 <wire x1="4.7625" y1="3.81" x2="4.7625" y2="11.0975" width="0.4064" layer="16"/>
 </signal>
-<signal name="QE">
+<signal name="SW">
 <contactref element="R12" pad="1"/>
 <contactref element="IC1" pad="4"/>
@@
 <wire x1="15.24" y1="15.5575" x2="15.24" y2="16.1775" width="0.4064" layer="16"/>
 </signal>
-<signal name="QF">
+<signal name="AUX_OK">
 <contactref element="R11" pad="1"/>
 <contactref element="IC1" pad="5"/>
@@
 <wire x1="10.175" y1="28.56" x2="9.525" y2="28.56" width="0.4064" layer="16"/>
 </signal>
-<signal name="QG">
+<signal name="NW">
 <contactref element="R10" pad="1"/>
 <contactref element="IC1" pad="6"/>
@@
 <wire x1="13.97" y1="29.21" x2="14.9075" y2="29.21" width="0.4064" layer="16"/>
 </signal>
-<signal name="QH">
+<signal name="W">
 <contactref element="R9" pad="1"/>
 <contactref element="IC1" pad="7"/>
@@
 <wire x1="13.97" y1="14.9225" x2="13.97" y2="19.035" width="0.4064" layer="16"/>
 </signal>
-<signal name="Q0">
+<signal name="S">
 <contactref element="R1" pad="1"/>
 <contactref element="IC2" pad="15"/>
@@
 <wire x1="26.4166" y1="11.785" x2="26.4541" y2="11.7475" width="0.4064" layer="16"/>
 </signal>
-<signal name="Q1">
+<signal name="E">
 <contactref element="R2" pad="1"/>
 <contactref element="IC2" pad="1"/>
@@
 <wire x1="32.6009" y1="13.8209" x2="32.6009" y2="13.0175" width="0.4064" layer="16"/>
 </signal>
-<signal name="Q2">
+<signal name="NE">
 <contactref element="R3" pad="1"/>
 <contactref element="IC2" pad="2"/>
@@
 <wire x1="34.465" y1="20.585" x2="34.465" y2="12.085" width="0.4064" layer="16"/>
 </signal>
-<signal name="Q3">
+<signal name="N">
 <contactref element="R4" pad="1"/>
 <contactref element="IC2" pad="3"/>
@@
 <wire x1="35.665" y1="21.485" x2="35.665" y2="11.385" width="0.4064" layer="16"/>
 </signal>
-<signal name="Q4">
+<signal name="SE">
 <contactref element="R5" pad="1"/>
 <contactref element="IC2" pad="4"/>
@@
 <wire x1="31.565" y1="14.985" x2="31.565" y2="15.77" width="0.4064" layer="16"/>
 </signal>
-<signal name="Q5">
+<signal name="SETUP">
 <contactref element="R6" pad="1"/>
 <contactref element="IC2" pad="5"/>
@@
 <wire x1="41.365" y1="10.6675" x2="41.335" y2="10.6975" width="0.4064" layer="16"/>
 </signal>
-<signal name="Q6">
+<signal name="MAG_CAL">
 <contactref element="R7" pad="1"/>
 <contactref element="IC2" pad="6"/>
@@
 <wire x1="36.52" y1="25.745" x2="36.52" y2="29.145" width="0.4064" layer="16"/>
 </signal>
-<signal name="Q7">
+<signal name="GYRO_CAL">
 <contactref element="R8" pad="1"/>
 <contactref element="IC2" pad="7"/>
