File: eagle/v3/murdock_mcu_v3.brd (EAGLE design)
At the start: 47 x 31.8 mm, 35 parts, among them IC1 MPU-9150, IC2 LT1763CS8-3.3, IC3 STM32F4XX_64, IC4 BMP085, IC5 24LC16BSN, T1 PFET, U1 USD-SOCKETNEW, X2 MURDOCK_STACK

Commit message: invert sbus
Parts:
- added R8: 1k, SparkFun-Resistors:0402-RES
- added R9: 10k, SparkFun-Resistors:0402-RES
- added T2: BC817, transistor:SOT23
Connections:
- new net N$11: IC3.17, R8.1, T2.3
- new net N$12: R9.1, T2.1
- net +3V3: now also R8.2
- net GND: now also T2.2
- net PWM2: now also R9.2; no longer IC3.17
Routing:
- net PWM2: track 69.2 -> 86.4 mm
- net N$11: track 0.00 -> 4.55 mm
- net +3V3: track 187.0 -> 190.0 mm, vias 9 -> 10
- net N$12: track 0.00 -> 1.37 mm
- net RX: track 14.7 -> 13.6 mm
- net PWM7: track 25.2 -> 25.9 mm
- net PPM: track 17.1 -> 16.4 mm
