File: eagle/v3/murdock_top_v3.brd (EAGLE design)
At the start: 47 x 31.8 mm, 35 parts, among them IC1 74HC595D, IC2 74HC595D, X1 MURDOCK_STACK

Commit message: final touches
Parts:
- moved R16 0.45 mm to (39.3, 18.8)
Changed lines of the file:
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@@
 <layer number="20" name="Dimension" color="15" fill="1" visible="yes" active="yes"/>
 <layer number="21" name="tPlace" color="7" fill="1" visible="yes" active="yes"/>
-<layer number="22" name="bPlace" color="7" fill="1" visible="no" active="yes"/>
+<layer number="22" name="bPlace" color="7" fill="1" visible="yes" active="yes"/>
 <layer number="23" name="tOrigins" color="15" fill="1" visible="yes" active="yes"/>
-<layer number="24" name="bOrigins" color="15" fill="1" visible="no" active="yes"/>
+<layer number="24" name="bOrigins" color="15" fill="1" visible="yes" active="yes"/>
 <layer number="25" name="tNames" color="14" fill="1" visible="yes" active="yes"/>
 <layer number="26" name="bNames" color="7" fill="1" visible="no" active="yes"/>
@@
 <attribute name="VALUE" x="7.997" y="18.698" size="0.4064" layer="28" rot="MR90"/>
 </element>
-<element name="R16" library="SparkFun-Passives" package="0402-RES" value="150R" x="39.305" y="18.3183" smashed="yes" rot="MR90">
-<attribute name="NAME" x="37.6035" y="17.2293" size="0.8128" layer="26" font="vector" ratio="10" rot="MR90"/>
-<attribute name="VALUE" x="38.162" y="17.2388" size="0.4064" layer="28" rot="MR90"/>
+<element name="R16" library="SparkFun-Passives" package="0402-RES" value="150R" x="39.305" y="18.7683" smashed="yes" rot="MR90">
+<attribute name="NAME" x="37.6035" y="17.6793" size="0.8128" layer="26" font="vector" ratio="10" rot="MR90"/>
+<attribute name="VALUE" x="38.162" y="17.6888" size="0.4064" layer="28" rot="MR90"/>
 </element>
 <element name="X1" library="murdock" package="MURDOCK_STACK" value="MURDOCK_STACK" x="0" y="0" smashed="yes"/>
@@
 <wire x1="39.065" y1="2.285" x2="39.065" y2="10.385" width="0.4064" layer="1"/>
 <wire x1="39.065" y1="10.385" x2="37.515" y2="11.935" width="0.4064" layer="1"/>
-<wire x1="37.515" y1="11.935" x2="37.5158" y2="15.247" width="0.4064" layer="1"/>
-<via x="38.695" y="16.4262" extent="1-16" drill="0.4"/>
-<wire x1="37.5158" y1="15.247" x2="38.695" y2="16.4262" width="0.4064" layer="1"/>
-<wire x1="39.305" y1="17.6683" x2="39.3288" y2="17.0608" width="0.4064" layer="16"/>
-<wire x1="39.3288" y1="17.0608" x2="38.695" y2="16.4262" width="0.4064" layer="16"/>
+<wire x1="37.515" y1="11.935" x2="37.5158" y2="15.747" width="0.4064" layer="1"/>
+<via x="38.695" y="16.9262" extent="1-16" drill="0.4"/>
+<wire x1="37.5158" y1="15.747" x2="38.695" y2="16.9262" width="0.4064" layer="1"/>
+<wire x1="39.305" y1="18.1183" x2="39.305" y2="17.5362" width="0.4064" layer="16"/>
+<wire x1="39.305" y1="17.5362" x2="38.695" y2="16.9262" width="0.4064" layer="16"/>
 </signal>
 <signal name="QB">
@@
 <contactref element="R16" pad="2"/>
 <contactref element="LED1" pad="K"/>
-<wire x1="39.305" y1="18.9683" x2="39.305" y2="20.9744" width="0.4064" layer="16"/>
+<wire x1="39.305" y1="19.4183" x2="39.305" y2="20.9744" width="0.4064" layer="16"/>
 <wire x1="39.305" y1="20.9744" x2="39.165" y2="21.0058" width="0.4064" layer="16"/>
 </signal>
@@
 <contactref element="LED9" pad="A"/>
 <wire x1="5.165" y1="31.135" x2="18.1080875" y2="31.135" width="0.4064" layer="16"/>
-<via x="30.465" y="25.785" extent="1-16" drill="0.4"/>
-<wire x1="30.465" y1="25.785" x2="35.465" y2="30.785" width="0.4064" layer="1"/>
-<via x="35.465" y="30.785" extent="1-16" drill="0.4"/>
-<wire x1="35.465" y1="30.785" x2="35.815" y2="31.135" width="0.4064" layer="16"/>
-<wire x1="35.815" y1="31.135" x2="42.565" y2="31.135" width="0.4064" layer="16"/>
+<via x="31.065" y="25.085" extent="1-16" drill="0.4"/>
+<wire x1="31.065" y1="25.085" x2="36.415" y2="30.435" width="0.4064" layer="1"/>
+<via x="36.415" y="30.435" extent="1-16" drill="0.4"/>
+<wire x1="36.415" y1="30.435" x2="37.115" y2="31.135" width="0.4064" layer="16"/>
+<wire x1="37.115" y1="31.135" x2="42.565" y2="31.135" width="0.4064" layer="16"/>
 <wire x1="42.565" y1="31.135" x2="43.165" y2="30.535" width="0.4064" layer="16"/>
 <wire x1="43.165" y1="30.535" x2="42.765" y2="29.21" width="0.4064" layer="16"/>
@@
 <wire x1="21.3205875" y1="27.585" x2="21.2080875" y2="27.585" width="0.4064" layer="16"/>
 <wire x1="21.695" y1="29.385" x2="21.695" y2="27.585" width="0.4064" layer="16"/>
-<wire x1="30.465" y1="25.785" x2="29.24559375" y2="24.56559375" width="0.4064" layer="16"/>
-<wire x1="29.24559375" y1="24.56559375" x2="28.61559375" y2="24.56559375" width="0.4064" layer="16"/>
+<wire x1="31.065" y1="25.085" x2="30.54559375" y2="24.56559375" width="0.4064" layer="16"/>
+<wire x1="30.54559375" y1="24.56559375" x2="28.61559375" y2="24.56559375" width="0.4064" layer="16"/>
 <wire x1="4.365" y1="30.335" x2="5.165" y2="31.135" width="0.4064" layer="16"/>
 <wire x1="19.79779375" y1="26.06220625" x2="21.3205875" y2="27.585" width="0.4064" layer="16"/>
@@
 </signal>
 </signals>
-<errors>
-</errors>
 </board>
 </drawing>
